File: pcb/prototype/soth-core.sch (EAGLE design)
At the start: 22 parts, among them IC1 AE-FT231X(FT231X) USB-Serial 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, IC2 REG1117, IC3 TC7SZ125F, IC4 TC7SZ125F, IC5 12113(LPS331AP) Pressure Sens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, U1 ATXMEGA32D4-AU, X1 5V/4A

Commit message: Created v0.1
Parts:
- removed X1: 5V/4A, con-conrad:733980-62
- added H1, H2: MOUNT-HOLE3.0, holes:MOUNT-HOLE3.0
- added SV7: PowerSupply, con-amp-mt:S02P
Connections:
- net +3V3: now also IC5.5
- net +5V: now also SV7-1.S; no longer X1.2, X1.3
- net GND: now also IC5.4, SV7-2.S; no longer X1.1
Other:
- moved on the sheet: IC5
