File: pcb/v0.1/core/soth-core.sch (EAGLE design)
At the start: 31 parts, among them IC1 ATXMEGA32E5-AU, M1 SMALL_SERVO, M2 SMALL_SERVO, M3 SMALL_SERVO, M4 SMALL_SERVO, M5 SMALL_SERVO, U1 LDO-TPS78233

Commit message: Bugfix pcb design. Replace LDO parts.
Parts:
- removed U1: LDO-TPS78233, SparkFun-PowerIC:LDO-TPS78233
- added C3: 0u01, rcl:C-EUC1608
- added IC2: TPS77001, texas:TPS77001
Connections:
- new net N$25: C3.1, IC2.NC/FB
- net +3V3: now also IC2.OUT; no longer U1.VCC
- net +5V: now also IC2.IN; no longer U1.IN
- net GND: now also IC2.GND; no longer U1.GND
- net GNDA: now also C3.2
- net N$2: now also IC2.!EN; no longer U1.EN
Other:
- moved on the sheet: C2, R1
Changed lines of the file:
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@@
 <part name="P+2" library="supply1" deviceset="+5V" device=""/>
 <part name="CN1" library="SparkFun-Connectors" deviceset="M03" device="PTH"/>
-<part name="U1" library="SparkFun-PowerIC" deviceset="LDO-TPS78233" device=""/>
 <part name="C1" library="rcl" deviceset="C-EU" device="C1608" value="0u1"/>
 <part name="C2" library="rcl" deviceset="C-EU" device="C1608" value="1u"/>
@@
 <part name="GND11" library="supply1" deviceset="GNDA" device="" value="GND3V3"/>
 <part name="U$2" library="Soth" deviceset="SOTH_LOGO" device=""/>
+<part name="IC2" library="texas" deviceset="TPS770*" device="" technology="01"/>
+<part name="C3" library="rcl" deviceset="C-EU" device="C1608" value="0u01"/>
+<part name="GND12" library="supply1" deviceset="GNDA" device="" value="GND3V3"/>
 </parts>
 <sheets>
@@
 <instance part="GND2" gate="1" x="71.12" y="116.84"/>
 <instance part="GND3" gate="1" x="66.04" y="68.58"/>
-<instance part="GND4" gate="1" x="129.54" y="119.38"/>
+<instance part="GND4" gate="1" x="144.78" y="114.3"/>
 <instance part="+3V1" gate="G$1" x="73.66" y="109.22"/>
-<instance part="+3V2" gate="G$1" x="129.54" y="147.32"/>
+<instance part="+3V2" gate="G$1" x="144.78" y="147.32"/>
 <instance part="P+1" gate="1" x="71.12" y="147.32"/>
 <instance part="P+2" gate="1" x="40.64" y="119.38"/>
 <instance part="CN1" gate="G$1" x="58.42" y="137.16"/>
-<instance part="U1" gate="G$1" x="114.3" y="132.08"/>
 <instance part="C1" gate="G$1" x="76.2" y="132.08"/>
-<instance part="C2" gate="G$1" x="129.54" y="132.08"/>
-<instance part="R1" gate="G$1" x="96.52" y="127"/>
+<instance part="C2" gate="G$1" x="144.78" y="132.08"/>
+<instance part="R1" gate="G$1" x="96.52" y="132.08"/>
 <instance part="GND5" gate="1" x="243.84" y="33.02"/>
 <instance part="+3V3" gate="G$1" x="193.04" y="106.68"/>
@@
 <instance part="GND11" gate="1" x="88.9" y="12.7"/>
 <instance part="U$2" gate="G$1" x="228.6" y="17.78"/>
+<instance part="IC2" gate="G$1" x="114.3" y="132.08"/>
+<instance part="C3" gate="G$1" x="132.08" y="124.46"/>
+<instance part="GND12" gate="1" x="132.08" y="114.3"/>
 </instances>
 <busses>
@@
 <wire x1="71.12" y1="121.92" x2="76.2" y2="121.92" width="0.1524" layer="91"/>
 <wire x1="76.2" y1="121.92" x2="76.2" y2="127" width="0.1524" layer="91"/>
-<wire x1="76.2" y1="121.92" x2="86.36" y2="121.92" width="0.1524" layer="91"/>
-<wire x1="86.36" y1="121.92" x2="86.36" y2="132.08" width="0.1524" layer="91"/>
-<pinref part="U1" gate="G$1" pin="GND"/>
-<wire x1="86.36" y1="132.08" x2="104.14" y2="132.08" width="0.1524" layer="91"/>
+<wire x1="76.2" y1="121.92" x2="88.9" y2="121.92" width="0.1524" layer="91"/>
+<wire x1="88.9" y1="121.92" x2="88.9" y2="127" width="0.1524" layer="91"/>
 <junction x="76.2" y="121.92"/>
 <junction x="71.12" y="121.92"/>
+<pinref part="IC2" gate="G$1" pin="GND"/>
+<wire x1="88.9" y1="127" x2="104.14" y2="127" width="0.1524" layer="91"/>
 </segment>
 <segment>
@@
 <pinref part="C2" gate="G$1" pin="2"/>
 <pinref part="GND4" gate="1" pin="GNDA"/>
-<wire x1="129.54" y1="127" x2="129.54" y2="121.92" width="0.1524" layer="91"/>
+<wire x1="144.78" y1="127" x2="144.78" y2="116.84" width="0.1524" layer="91"/>
 </segment>
 <segment>
@@
 <wire x1="88.9" y1="20.32" x2="96.52" y2="20.32" width="0.1524" layer="91"/>
 </segment>
+<segment>
+<pinref part="C3" gate="G$1" pin="2"/>
+<wire x1="132.08" y1="116.84" x2="132.08" y2="119.38" width="0.1524" layer="91"/>
+<pinref part="GND12" gate="1" pin="GNDA"/>
+</segment>
 </net>
 <net name="+3V3" class="3">
@@
 </segment>
 <segment>
-<wire x1="121.92" y1="137.16" x2="129.54" y2="137.16" width="0.1524" layer="91"/>
-<wire x1="129.54" y1="137.16" x2="129.54" y2="144.78" width="0.1524" layer="91"/>
+<wire x1="127" y1="137.16" x2="144.78" y2="137.16" width="0.1524" layer="91"/>
+<wire x1="144.78" y1="137.16" x2="144.78" y2="144.78" width="0.1524" layer="91"/>
 <pinref part="+3V2" gate="G$1" pin="+3V3"/>
-<pinref part="U1" gate="G$1" pin="VCC"/>
 <pinref part="C2" gate="G$1" pin="1"/>
-<wire x1="129.54" y1="137.16" x2="129.54" y2="134.62" width="0.1524" layer="91"/>
-<junction x="129.54" y="137.16"/>
+<wire x1="144.78" y1="137.16" x2="144.78" y2="134.62" width="0.1524" layer="91"/>
+<junction x="144.78" y="137.16"/>
+<pinref part="IC2" gate="G$1" pin="OUT"/>
 </segment>
 <segment>
@@
 <wire x1="66.04" y1="137.16" x2="71.12" y2="137.16" width="0.1524" layer="91"/>
 <wire x1="71.12" y1="137.16" x2="71.12" y2="144.78" width="0.1524" layer="91"/>
-<wire x1="104.14" y1="137.16" x2="88.9" y2="137.16" width="0.1524" layer="91"/>
 <junction x="71.12" y="137.16"/>
 <pinref part="P+1" gate="1" pin="+5V"/>
 <pinref part="CN1" gate="G$1" pin="2"/>
-<pinref part="U1" gate="G$1" pin="IN"/>
 <pinref part="C1" gate="G$1" pin="1"/>
 <wire x1="88.9" y1="137.16" x2="76.2" y2="137.16" width="0.1524" layer="91"/>
 <wire x1="76.2" y1="137.16" x2="71.12" y2="137.16" width="0.1524" layer="91"/>
 <wire x1="76.2" y1="134.62" x2="76.2" y2="137.16" width="0.1524" layer="91"/>
+<wire x1="88.9" y1="132.08" x2="88.9" y2="137.16" width="0.1524" layer="91"/>
+<junction x="76.2" y="137.16"/>
 <pinref part="R1" gate="G$1" pin="1"/>
-<wire x1="91.44" y1="127" x2="88.9" y2="127" width="0.1524" layer="91"/>
-<wire x1="88.9" y1="127" x2="88.9" y2="137.16" width="0.1524" layer="91"/>
-<junction x="76.2" y="137.16"/>
+<wire x1="88.9" y1="132.08" x2="91.44" y2="132.08" width="0.1524" layer="91"/>
+<pinref part="IC2" gate="G$1" pin="IN"/>
+<wire x1="104.14" y1="137.16" x2="88.9" y2="137.16" width="0.1524" layer="91"/>
 <junction x="88.9" y="137.16"/>
 </segment>
@@
 </segment>
 </net>
-<net name="N$2" class="0">
-<segment>
-<pinref part="R1" gate="G$1" pin="2"/>
-<wire x1="101.6" y1="127" x2="104.14" y2="127" width="0.1524" layer="91"/>
-<pinref part="U1" gate="G$1" pin="EN"/>
-</segment>
-</net>
 <net name="N$4" class="0">
 <segment>
@@
 </segment>
 </net>
+<net name="N$2" class="0">
+<segment>
+<pinref part="R1" gate="G$1" pin="2"/>
+<pinref part="IC2" gate="G$1" pin="!EN"/>
+<wire x1="101.6" y1="132.08" x2="104.14" y2="132.08" width="0.1524" layer="91"/>
+</segment>
+</net>
+<net name="N$25" class="0">
+<segment>
+<pinref part="IC2" gate="G$1" pin="NC/FB"/>
+<pinref part="C3" gate="G$1" pin="1"/>
+<wire x1="127" y1="127" x2="132.08" y2="127" width="0.1524" layer="91"/>
+</segment>
+</net>

Commit message: Change microcontroller from atxmega32d4 to atxmega32e5
Parts:
- LED1: value RED CONNECT -> GREEN CONNECTED
- LED2: value GREEN CONNECTED -> RED CONNECT
- LED3: value GREEN STATUS -> YELLOW STATUS
- R2, R3, R7: value 1k -> 2k
Connections:
- new net N$26: IC1.PC2, U$1.RESET
Other:
- moved on the sheet: H1, H2, LED1, LED2, R2, R3, R4, R5, T1, T2, T3
