File: pcb/v0.1/extension/soth-ext.sch (EAGLE design)
At the start: 5 parts, among them IC1 MPU-9250, IC2 BME280

Commit message: Successfully gps data rcv.
Connections:
- net N$3: now also U$1.P$3; no longer U$1.P$4
Changed lines of the file:
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@@
 <pinref part="JP1" gate="G$1" pin="5"/>
 <wire x1="20.32" y1="33.02" x2="53.34" y2="33.02" width="0.1524" layer="91"/>
-<wire x1="53.34" y1="33.02" x2="53.34" y2="27.94" width="0.1524" layer="91"/>
-<pinref part="U$1" gate="G$1" pin="P$4"/>
-<wire x1="53.34" y1="27.94" x2="60.96" y2="27.94" width="0.1524" layer="91"/>
+<wire x1="53.34" y1="33.02" x2="53.34" y2="25.4" width="0.1524" layer="91"/>
+<pinref part="U$1" gate="G$1" pin="P$3"/>
+<wire x1="53.34" y1="25.4" x2="60.96" y2="25.4" width="0.1524" layer="91"/>
 </segment>
 </net>
